File: hardware/version 2011-2017/KiCad/SAW30_v2011-2017_original1Layer_THT.kicad_pcb (KiCad board)
At the start: 2 copper layers, 142 x 95 mm, 157 parts, among them J1 +UB, J10 OUT1, J11 OUT1_0, J12 OUT2, J13 OUT2_0, J14 OUT3, J15 OUT3_0, J16 OUT4, J17 OUT4_0, J2 UB 0 (GND), J3 -UB, J4 IN1 +, J5 IN1 0 (GND), J6 IN1 -, J7 IN2 +, J8 IN2 0 (GND), J9 IN2 -, P1 5k, P11 5k, P2 5k, P21 5k, P3 5k, P31 5k, P4 5k, P41 5k, P5 10k, P6 10k, Q1 TIP137, Q2 TIP132, SW1 DRS4010, SW2 DRS4010, SW3 DRS4010, SW4 DRS4010, SW5 DRS4010, SW6 DRS4010, SW7 DRS4010, SW8 DRS4010, U1 MC33079, U2 MC33079, U3 MC33079, U4 MC33079

Commit message: Add files via upload
Parts:
- C1, C2, C3, C4, C5, C6, C7, C8: footprint analoghifi:C_Multi_THT_1-Layer_alternative_2 -> analoghifi:C_Multi_THT_1-Layer_alternative_2_EMZ
- C10, C9: footprint Connector_PinSocket_2.54mm:PinSocket_1x05_P2.54mm_Vertical -> analoghifi:Preci-Dip_1x05_P2.54mm_Vertical_no_silk
- C11, C12: footprint analoghifi:CP_Radial_D10.0mm_P5.00mm_minmal_silk -> analoghifi:CP_Radial_D10.0mm_H12.5mm_P5.00mm_minmal_silk
- C13, C14, C15, C16: footprint analoghifi:CP_Radial_D8.0mm_P3.50mm_minimal_silk -> analoghifi:CP_Radial_Black_D8.2mm_H12.5mm_P3.50mm_minimal_silk
- moved P31 2.84 mm to (179.3, 55.5)
- moved P11 2.55 mm to (119.0, 55.5)
- moved P41 2.55 mm to (207.0, 55.5)
- moved P21 2.26 mm to (146.7, 55.5)
- moved P3 0.66 mm to (190.7, 63.0)
- moved R39 0.56 mm to (212.2, 66.6)
- moved R40 0.56 mm to (212.2, 61.0)
- moved R70 0.56 mm to (202.0, 63.5)
- moved P4 0.46 mm to (218.5, 63.0)
- moved P1 0.46 mm to (102.5, 63.0)
- moved J10 0.40 mm to (108.0, 52.0)
- moved J11 0.40 mm to (102.0, 52.0)
- moved J16 0.40 mm to (224.0, 52.0)
- moved J17 0.40 mm to (218.0, 52.0)
- moved R19 0.36 mm to (124.0, 66.6)
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Routing:
- net Net-(J10-Pad1): track 34.1 -> 35.4 mm
- net Net-(J16-Pad1): track 34.2 -> 35.2 mm
- net Net-(J14-Pad1): track 51.8 -> 52.6 mm
- net Net-(P3-Pad3): track 29.4 -> 30.0 mm
- net HP2 out: track 70.1 -> 70.7 mm
