File: hardware/version 2011-2017/KiCad/SAW30_v2011-2017_original1Layer_THT.kicad_sch (KiCad schematic)
At the start: 153 parts, among them J1 +UB, J10 OUT1, J11 OUT1_0, J12 OUT2, J13 OUT2_0, J14 OUT3, J15 OUT3_0, J16 OUT4, J17 OUT4_0, J2 UB 0 (GND), J3 -UB, J4 IN1 +, J5 IN1 0 (GND), J6 IN1 -, J7 IN2 +, J8 IN2 0 (GND), J9 IN2 -, P1 5k, P11 5k, P2 5k, P21 5k, P3 5k, P31 5k, P4 5k, P41 5k, P5 10k, P6 10k, Q1 TIP137, Q2 TIP132, SW1 DRS4010, SW2 DRS4010, SW3 DRS4010, SW4 DRS4010, SW5 DRS4010, SW6 DRS4010, SW7 DRS4010, SW8 DRS4010, U1 MC33079, U2 MC33079, U3 MC33079, U4 MC33079

Commit message: Add files via upload
Parts:
- C1, C2, C3, C4, C5, C6, C7, C8: footprint analoghifi:C_Multi_THT_1-Layer_alternative_2 -> analoghifi:C_Multi_THT_1-Layer_alternative_2_EMZ
- C10, C9: value 680nF -> (none); footprint Connector_PinSocket_2.54mm:PinSocket_1x05_P2.54mm_Vertical -> (none)
- C11, C12: footprint analoghifi:CP_Radial_D10.0mm_P5.00mm_minmal_silk -> analoghifi:CP_Radial_D10.0mm_H12.5mm_P5.00mm_minmal_silk
- C13, C14, C15, C16: footprint analoghifi:CP_Radial_D8.0mm_P3.50mm_minimal_silk -> analoghifi:CP_Radial_Black_D8.2mm_H12.5mm_P3.50mm_minimal_silk
