File: hardware/version 07.2017 until now/KiCad/SAW30_original_1Layer_THT.kicad_sch (KiCad schematic)
At the start: 151 parts, among them J1 +UB, J10 OUT1, J11 OUT1_0, J12 OUT2, J13 OUT2_0, J14 OUT3, J15 OUT3_0, J16 OUT4, J17 OUT4_0, J2 UB 0 (GND)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

Commit message: Add files via upload
Parts:
- C10, C11, C12, C9: value 220uF/35V -> (none); footprint analoghifi:CP_Radial_D8.0mm_P3.50mm_minimal_silk -> (none)
